File: Electronics/teensiPCB.kicad_pcb (KiCad board)
At the start: 2 copper layers, 45 x 84 mm, 15 parts, among them J1 screw terminal, J2 Conn_01x02, J5 UART1, J6 UART2, J7 I2C ext, SW1 SW_Push, U2 SAM-M10Q-00B

Commit message: PCB redesign 0.1
Parts:
- moved J6 11.2 mm to (180.5, 91.4), turned to 0 degrees
- moved J5 7.21 mm to (180.2, 83.5), turned to 0 degrees
- moved J7 6.95 mm to (180.2, 73.7), turned to 0 degrees
Routing:
- net +3V3: track 135.2 -> 0.00 mm
- net Net-(U2-SDA): track 90.0 -> 0.00 mm, vias 1 -> 0
- net Net-(U2-SCL): track 77.7 -> 0.00 mm, vias 1 -> 0
- net Net-(J7-Pin_3): track 42.1 -> 0.00 mm
- net Net-(U2-RESET_N): track 41.6 -> 0.00 mm, vias 1 -> 0
- net Net-(J7-Pin_2): track 36.3 -> 0.00 mm
- net Net-(J5-Pin_2): track 24.8 -> 0.00 mm
- net Net-(J6-Pin_2): track 22.2 -> 0.00 mm
- net GND: track 21.6 -> 0.00 mm, vias 11 -> 0
- net Net-(J5-Pin_3): track 18.7 -> 0.00 mm
- net Net-(J6-Pin_3): track 16.0 -> 0.00 mm
- net Net-(J1-Pin_1): track 9.44 -> 0.00 mm
- net Net-(C1-Pad1): track 4.52 -> 0.00 mm

Commit message: Updated TODOs
Parts:
- removed J6: UART2, Connector_JST:JST_XH_B4B-XH-A_1x04_P2.50mm_Vertical
- removed J7: I2C ext, Connector_JST:JST_XH_B4B-XH-A_1x04_P2.50mm_Vertical
- added UART3: Conn_01x02, Connector_JST:JST_XH_B2B-XH-A_1x02_P2.50mm_Vertical, F.Cu at (183.6, 92.9)
- moved Ue1 34.5 mm to (240.8, 89.0)
- moved J5 1.00 mm to (179.7, 82.7)
Connections:
- Ue1 pad 10: Net-(J6-Pin_3) -> TX_OUT_MOTOR1
- Ue1 pad 16: Net-(J7-Pin_2) -> SCL_OUT_MOTOR2
- Ue1 pad 17: Net-(J7-Pin_3) -> SDA_OUT_MOTOR2
- Ue1 pad 42: (no net) -> TX_TO_GCS
- Ue1 pad 43: unconnected-(Ue1-GND-Pad34) -> RX_TO_GCS
- Ue1 pad 44: GND -> unconnected-(Ue1-PWM-Pad44)
- Ue1 pad 45: +3V3 -> unconnected-(Ue1-PWM-Pad45)
- Ue1 pad 9: Net-(J6-Pin_2) -> RX_OUT_MOTOR1
Routing:
- removed copper zone on B.Cu, net GND

Commit message: Change teensy symbol and footprint
Parts:
- added IC**: TEENSY41, Footprints:TEENSY41, F.Cu at (214.0, 114.5)
